File: $LIPO charger and Regulator.sch (KiCad schematic (older format))
At the start: 28 parts, among them CON1 USB-MICRO-B, P1 LIPO battery, P2 1.8V Regulator, P3 3.3V Regulator, U1 LTC3558

Commit message: Modified for 5.1V
Parts:
- CON1: footprint Connect:USB_Micro-B -> EE library:USB_Micro-B_SMD
- P2, P3: footprint Connect:bornier2 -> Connect:PINHEAD1-2
- R14: footprint Resistors_SMD:R_0603_HandSoldering -> Resistors_SMD:R_0603
Changed lines of the file:
@@
 F 0 "CON1" H 2400 1950 50  0000 C CNN
 F 1 "USB-MICRO-B" H 2550 1250 50  0000 C CNN
-F 2 "Connect:USB_Micro-B" H 2700 1500 50  0001 C CNN
+F 2 "EE library:USB_Micro-B_SMD" H 2700 1500 50  0001 C CNN
 F 3 "" H 2700 1500 50  0000 C CNN
 	1    2700 1600
@@
 F 0 "P2" H 8900 2750 50  0000 C CNN
 F 1 "1.8V Regulator" H 9250 2600 50  0000 C CNN
-F 2 "Connect:bornier2" H 8900 2600 60  0001 C CNN
+F 2 "Connect:PINHEAD1-2" H 8900 2600 60  0001 C CNN
 F 3 "" H 8900 2600 60  0000 C CNN
 	1    8900 2600
@@
 F 0 "P3" H 8950 4500 50  0000 C CNN
 F 1 "3.3V Regulator" H 9300 4350 50  0000 C CNN
-F 2 "Connect:bornier2" H 8950 4350 60  0001 C CNN
+F 2 "Connect:PINHEAD1-2" H 8950 4350 60  0001 C CNN
 F 3 "" H 8950 4350 60  0000 C CNN
 	1    8950 4350
@@
 P 7650 3650
 F 0 "R14" V 7730 3650 50  0000 C CNN
-F 1 "15M" H 7900 3700 50  0000 C CNN
-F 2 "Resistors_SMD:R_0603_HandSoldering" V 7580 3650 30  0001 C CNN
+F 1 "15M" V 7650 3650 50  0000 C CNN
+F 2 "Resistors_SMD:R_0603" V 7580 3650 30  0001 C CNN
 F 3 "" H 7650 3650 30  0000 C CNN
 	1    7650 3650
