File: LIPO charger and Regulator.kicad_pcb (KiCad board)
At the start: 2 copper layers, 33.3 x 24 mm, 33 parts, among them CON1 USB-MICRO-B, P1 LIPO battery, P2 1.8V Regulator, P3 3.3V Regulator, U1 LTC3558

Commit message: legend
Parts:
- added JP1: JUMPER, Pin_Headers:Pin_Header_Straight_1x02, F.Cu at (135.9, 102.5)
- added P4: CONN_01X02, Pin_Headers:Pin_Header_Straight_1x02, F.Cu at (149.8, 104.7)
- LIPO : renamed from P1
- moved LIPO  3.30 mm to (146.5, 113.6)
- moved LOGO 1.22 mm to (145.1, 107.0)
- moved REF** 0.30 mm to (149.8, 118.5)
- turned D1 to 90 degrees
Connections:
- R2 pad 2: Net-(D1-Pad1) -> Net-(D1-Pad2)
- U1 pad 12: GND -> Net-(JP1-Pad2)
- U1 pad 19: Net-(D1-Pad2) -> Net-(D1-Pad1)
Routing:
- net Net-(JP1-Pad2): track 0.00 -> 29.6 mm, vias 0 -> 1
- net Net-(C1-Pad1): track 45.2 -> 22.2 mm, vias 4 -> 2
- net /BAT: track 41.5 -> 51.4 mm, vias 4 -> 3
- net GND: track 153.6 -> 147.4 mm, vias 1 -> 2
- net Net-(D1-Pad2): track 4.71 -> 1.80 mm
- net Net-(D1-Pad1): track 1.80 -> 4.71 mm
- net Net-(R1-Pad1): track 18.0 -> 17.0 mm
Other:
- outline, holes or cut-outs redrawn
- board text added: "+"
- board text added: "-"
- board text added: "BAT"
- board text added: "Buckster Ver 0.1"
