File: LIPO charger and Regulator.sch (KiCad schematic (older format))
At the start: 28 parts, among them CON1 USB-MICRO-B, P1 LIPO battery, P2 1.8V Regulator, P3 3.3V Regulator, U1 LTC3558

Commit message: Modified for 5.1V
Connections:
- net GND: now also CON1.7 (SHELL2), CON1.8 (SHELL3)
Changed lines of the file:
@@
 LIBS:memory
 LIBS:xilinx
+LIBS:special
 LIBS:microcontrollers
 LIBS:dsp
@@
 $EndComp
 Wire Wire Line
-	3200 1400 3200 2300
-Wire Wire Line
 	2200 1400 2050 1400
 Wire Wire Line
@@
 	1    0    0    -1
 $EndComp
+Wire Wire Line
+	3200 1400 3200 2300
+Connection ~ 3200 1500
+Connection ~ 3200 1700
 $EndSCHEMATC

Commit message: legend
Parts:
- added JP1: JUMPER, Pin_Headers:Pin_Header_Straight_1x02, symbol JUMPER
- added P4: CONN_01X02, Pin_Headers:Pin_Header_Straight_1x02, symbol CONN_01X02
- CON1: footprint Connect:USB_Micro-B -> EE library:USB_Micro-B_SMD
- P2, P3: footprint Connect:bornier2 -> Connect:PINHEAD1-2
- R14: footprint Resistors_SMD:R_0603_HandSoldering -> Resistors_SMD:R_0603
Connections:
- net BAT: now also P4.1 (P1)
- net GND: now also JP1.1, P4.2 (P2); no longer U1.12 (SUSP)
- net at U1.19 (CHRG): now also D1.1 (K); no longer D1.2 (A)
- net at R2.2: now also D1.2 (A); no longer D1.1 (K)
- new net: JP1.2, U1.12 (SUSP)
